Commit message: Reoriented to X-forward Y-left system

File: urdf/omniplatform.urdf (robot description, URDF)
Before this commit: robot omniplatform, 4 links, 3 joints
Joints:
- joint wheel1_axis: origin xyz=0 0.077647 0 rpy=0 0 0 -> xyz=0.077647 0 0 rpy=0 0 0
- joint wheel2_axis: origin xyz=${cos(2*pi/3)*0 - sin(2*pi/3)*0.077647} ${sin(2*pi/3)*0 + cos(2*pi/3)*0.077647} 0 rpy=0 0 ${2*pi/3} -> xyz=${cos(2*pi/3)*0.077647 - sin(2*pi/3)*0} ${sin(2*pi/3)*0.077647 + cos(2*pi/3)*0} 0 rpy=0 0 ${2*pi/3}
- joint wheel3_axis: origin xyz=${cos(2*pi/3*2)*0 - sin(2*pi/3*2)*0.077647} ${sin(2*pi/3*2)*0 + cos(2*pi/3*2)*0.077647} 0 rpy=0 0 ${2*pi/3*2} -> xyz=${cos(2*pi/3*2)*0.077647 - sin(2*pi/3*2)*0} ${sin(2*pi/3*2)*0.077647 + cos(2*pi/3*2)*0} 0 rpy=0 0 ${2*pi/3*2}

Commit message: Added mouse encoders

File: urdf/omniplatform.urdf (robot description, URDF)
Before this commit: robot omniplatform, 4 links, 3 joints
Links:
- added link mouse1; visual cylinder length=0.02 radius=0.005
- added link mouse2; visual cylinder length=0.02 radius=0.005
Joints:
- added joint mouse1_joint: type fixed, parent base_link, child mouse1, origin xyz=0 0.03 -0.025
- added joint mouse2_joint: type fixed, parent base_link, child mouse2, origin xyz=0 -0.03 -0.025

Commit message: 4 mice

File: urdf/omniplatform.urdf (robot description, URDF)
Before this commit: robot omniplatform, 6 links, 5 joints
Links:
- added link mouse3; visual cylinder length=0.02 radius=0.005
- added link mouse4; visual cylinder length=0.02 radius=0.005
Joints:
- added joint mouse3_joint: type fixed, parent base_link, child mouse3, origin xyz=0 -0.03 -0.025
- added joint mouse4_joint: type fixed, parent base_link, child mouse4, origin xyz=0 -0.09 -0.025
- joint mouse1_joint: origin xyz=0 0.03 -0.025 -> xyz=0 0.09 -0.025
- joint mouse2_joint: origin xyz=0 -0.03 -0.025 -> xyz=0 0.03 -0.025
